Commit message: added damping to actuated joints

File: src/avatar_description/urdf/avatar_description.xacro (robot description, xacro)
@@ -85,4 +85,5 @@
         <axis xyz="0 -1 0" />
         <limit lower="${-pi/2}" upper="${pi/2}" effort="100" velocity="20" />
+        <dynamics damping="1.0" />
     </joint>
     <link name="diff_1_top">
@@ -114,4 +115,5 @@
         <axis xyz="1 0 0" />
         <limit lower="${-pi/2}" upper="${pi/2}" effort="100" velocity="20" />
+        <dynamics damping="1.0" />
     </joint>
     <link name="arm_link_1">
@@ -143,4 +145,5 @@
         <axis xyz="0 1 0" />
         <limit lower="${-pi}" upper="${pi}" effort="100" velocity="20" />
+        <dynamics damping="1.0" />
     </joint>
     <link name="diff_2_top">
@@ -172,4 +175,5 @@
         <axis xyz="1 0 0" />
         <limit lower="${-pi/2}" upper="${pi/2}" effort="100" velocity="20" />
+        <dynamics damping="1.0" />
     </joint>
     <link name="arm_link_2">
@@ -201,4 +205,5 @@
         <axis xyz="0 1 0" />
         <limit lower="${-pi}" upper="${pi}" effort="100" velocity="20" />
+        <dynamics damping="1.0" />
     </joint>
     <!-- Create transmissions for each moveable joint -->
